File: PCB/Omamori.kicad_pcb (KiCad board)
At the start: 2 copper layers, 26 x 36 mm, 13 parts, among them J1 Conn_01x04_MountingPin, U1 BQ25504, U2 MSP430G2210ID

Commit message: Made changes to PCB.
Parts:
- removed C1: C, Capacitor_THT:C_Rect_L7.2mm_W2.5mm_P5.00mm_FKS2_FKP2_MKS2_MKP2
- removed J1: Conn_01x04_MountingPin, Connector_PinHeader_2.54mm:PinHeader_1x04_P2.54mm_Vertical
- added CSuper1: C, Capacitor_THT:C_Rect_L7.2mm_W2.5mm_P5.00mm_FKS2_FKP2_MKS2_MKP2, B.Cu at (180.0, 102.5)
- D9: value WS2812B -> SK6812
- U2: value MSP430G2210ID -> ATtiny13A-SSU
- moved D2 16.3 mm to (168.5, 100.0), turned to 0 degrees
- moved D4 16.3 mm to (180.0, 111.5), turned to 90 degrees
- moved D6 16.3 mm to (191.5, 100.0), turned to 180 degrees
- moved D8 16.3 mm to (180.0, 88.5), turned to 270 degrees
- moved D1 16.0 mm to (172.0, 92.0), turned to 315 degrees
- moved D3 16.0 mm to (172.0, 108.0), turned to 45 degrees
- moved D5 16.0 mm to (188.0, 108.0), turned to 135 degrees
- moved D7 16.0 mm to (188.0, 92.0), turned to 225 degrees
- moved U1 2.24 mm to (175.0, 88.0)
- turned D9 to 90 degrees
- turned U2 to 180 degrees
Connections:
- D9 pad 1: (no net) -> GND
- D9 pad 2: (no net) -> Net-(D9-Pad2)
- D9 pad 3: GND -> Net-(D9-Pad3)
- D9 pad 4: (no net) -> Net-(D9-Pad4)
- U1 pad 10: (no net) -> Net-(U1-Pad10)
- U1 pad 16: (no net) -> Net-(U1-Pad16)
- U1 pad 17: (no net) -> Net-(U1-Pad17)
- U1 pad 3: (no net) -> Net-(U1-Pad3)
- U1 pad 4: (no net) -> Net-(U1-Pad4)
- U1 pad 5: (no net) -> Net-(U1-Pad5)
- U1 pad 6: (no net) -> Net-(U1-Pad6)
- U1 pad 7: (no net) -> Net-(U1-Pad7)
- U1 pad 8: (no net) -> Net-(U1-Pad8)
- U1 pad 9: (no net) -> Net-(U1-Pad9)
- U2 pad 1: Net-(U1-Pad15) -> Net-(U2-Pad1)
- U2 pad 2: (no net) -> Net-(U2-Pad2)
- U2 pad 3: (no net) -> Net-(U2-Pad3)
- U2 pad 4: Net-(U1-Pad11) -> GND
- U2 pad 5: (no net) -> Net-(D9-Pad2)
- U2 pad 6: (no net) -> Net-(U1-Pad11)
- U2 pad 7: (no net) -> Net-(D9-Pad3)
- U2 pad 8: (no net) -> Net-(U1-Pad15)
Routing:
- net GND: track 0.00 -> 26.7 mm
- net Net-(CSuper1-Pad1): track 0.00 -> 15.0 mm
- net Net-(D5-Pad2): track 0.00 -> 8.92 mm
- net Net-(D1-Pad2): track 0.00 -> 8.92 mm
- net Net-(D7-Pad2): track 0.00 -> 8.92 mm
- net Net-(D3-Pad2): track 0.00 -> 8.92 mm
- net Net-(D6-Pad2): track 0.00 -> 8.65 mm
- net Net-(D2-Pad2): track 0.00 -> 8.65 mm
- net Net-(D4-Pad2): track 0.00 -> 8.65 mm
