File: PCB/Omamori.sch (KiCad schematic (older format))
At the start: 13 parts, among them J1 Conn_01x04_MountingPin, U1 BQ25504, U2 MSP430G2210ID

Commit message: Made changes to PCB.
Parts:
- removed D9: WS2812B, LED_SMD:LED_WS2812B_PLCC4_5.0x5.0mm_P3.2mm, symbol LED:WS2812B
- removed J1: Conn_01x04_MountingPin, Connector_PinHeader_2.54mm:PinHeader_1x04_P2.54mm_Vertical, symbol Connector_Generic_MountingPin:Conn_01x04_MountingPin
- removed U2: MSP430G2210ID, Package_SO:SOIC-8_3.9x4.9mm_P1.27mm, symbol MCU_Texas_MSP430:MSP430G2210ID
- added D9: SK6812, LED_SMD:LED_SK6812_PLCC4_5.0x5.0mm_P3.2mm, symbol LED:SK6812
- added U2: ATtiny13A-SSU, Package_SO:SOIC-8_3.9x4.9mm_P1.27mm, symbol MCU_Microchip_ATtiny:ATtiny13A-SSU
- renumbered C1 to CSuper1
Connections:
- net GND: now also D9.1 (VSS), U2.4 (GND)
- net at U1.11 (VBAT_OK): now also U2.6 (PB1)
- net at U1.15 (VSTOR): now also U2.8 (VCC)
- new net: D9.2 (DIN), U2.5 (PB0)
- new net: D9.3 (VDD), U2.7 (PB2)
- no-connect marks 0 -> 1
Other:
- moved on the sheet: CSuper1, D1, D2, D3, D4, D5, D6, D7, D8, U1
