File: 0.2/Hardware/PCB_0.2.1/Omamori.sch (KiCad schematic (older format))
At the start: 34 parts, among them J1 Conn_01x04_Female, Q1 IRLML0030, U1 BQ25504, U2 TPS61222DCK, U3 ATtiny85, U4 TS-1233

Commit message: V3 update.
Parts:
- C_hvr1: footprint Capacitor_SMD:C_0603_1608Metric_Pad1.05x0.95mm_HandSolder -> Capacitor_SMD:C_0805_2012Metric_Pad1.18x1.45mm_HandSolder
- R_oc2: value 3.9M -> 4.3M
- R_ov1: value 6.8M -> 6.2M
- renumbered R_vdiv_1 to R_oc3, R_vdiv_2_1 to R_oc4, R_vdiv_2_2 to R_oc5
Changed lines of the file:
@@
 F 0 "C_hvr1" H 2615 2246 50  0000 L CNN
 F 1 "4.7uF" H 2615 2155 50  0000 L CNN
-F 2 "Capacitor_SMD:C_0603_1608Metric_Pad1.05x0.95mm_HandSolder" H 2538 2050 50  0001 C CNN
+F 2 "Capacitor_SMD:C_0805_2012Metric_Pad1.18x1.45mm_HandSolder" H 2538 2050 50  0001 C CNN
 F 3 "~" H 2500 2200 50  0001 C CNN
 	1    2500 2200
@@
 P 3050 2300
 F 0 "R_oc2" H 3120 2346 50  0000 L CNN
-F 1 "3.9M" H 3120 2255 50  0000 L CNN
+F 1 "4.3M" H 3120 2255 50  0000 L CNN
 F 2 "Resistor_SMD:R_0603_1608Metric_Pad1.05x0.95mm_HandSolder" V 2980 2300 50  0001 C CNN
 F 3 "~" H 3050 2300 50  0001 C CNN
@@
 P 2200 4150
 F 0 "R_ov1" H 2270 4196 50  0000 L CNN
-F 1 "6.8M" H 2270 4105 50  0000 L CNN
+F 1 "6.2M" H 2270 4105 50  0000 L CNN
 F 2 "Resistor_SMD:R_0603_1608Metric_Pad1.05x0.95mm_HandSolder" V 2130 4150 50  0001 C CNN
 F 3 "~" H 2200 4150 50  0001 C CNN
@@
 	5850 3700 5900 3700
 $Comp
-L Device:R R_vdiv_1
+L Device:R R_oc3
 U 1 1 61C235D3
 P 7650 1800
-F 0 "R_vdiv_1" H 7720 1846 50  0000 L CNN
+F 0 "R_oc3" H 7720 1846 50  0000 L CNN
 F 1 "1.8M" H 7720 1755 50  0000 L CNN
 F 2 "Resistor_SMD:R_0603_1608Metric_Pad0.98x0.95mm_HandSolder" V 7580 1800 50  0001 C CNN
@@
 $EndComp
 $Comp
-L Device:R R_vdiv_2_2
+L Device:R R_oc5
 U 1 1 61C24BDB
 P 7950 2300
-F 0 "R_vdiv_2_2" H 8020 2346 50  0000 L CNN
+F 0 "R_oc5" H 8020 2346 50  0000 L CNN
 F 1 "10M" H 8020 2255 50  0000 L CNN
 F 2 "Resistor_SMD:R_0603_1608Metric_Pad0.98x0.95mm_HandSolder" V 7880 2300 50  0001 C CNN
@@
 $EndComp
 $Comp
-L Device:R R_vdiv_2_1
+L Device:R R_oc4
 U 1 1 61C266D9
 P 7950 2000
-F 0 "R_vdiv_2_1" H 8020 2046 50  0000 L CNN
+F 0 "R_oc4" H 8020 2046 50  0000 L CNN
 F 1 "8.2M" H 8020 1955 50  0000 L CNN
 F 2 "Resistor_SMD:R_0603_1608Metric_Pad0.98x0.95mm_HandSolder" V 7880 2000 50  0001 C CNN
