File: 0.3/Hardware/PCB_0.3.0/Omamori.kicad_sch (KiCad schematic)
At the start: 28 parts, among them J1 Conn_01x04_Female, U1 BQ25570, U2 ATtiny85-20S, U3 TS-1233

Commit message: Voltage measurement update.
Parts:
- removed R_pulldown1: 10M, Resistor_SMD:R_0603_1608Metric_Pad1.05x0.95mm_HandSolder, symbol Device:R
- added R_VDIV1_1: 8.5M, Resistor_SMD:R_0603_1608Metric_Pad0.98x0.95mm_HandSolder, symbol Device:R
- added R_VDIV1_2: 10M, Resistor_SMD:R_0603_1608Metric_Pad0.98x0.95mm_HandSolder, symbol Device:R
- added R_VDIV2: 9M, Resistor_SMD:R_0603_1608Metric_Pad0.98x0.95mm_HandSolder, symbol Device:R
- L_bst1, L_bst2: footprint Inductor_SMD:L_Wuerth_MAPI-3015 -> Inductor_SMD:L_Taiyo-Yuden_NR-30xx_HandSoldering
Connections:
- net GND: now also R_VDIV2.2
- net Reset: now also R_VDIV1_1.1, R_VDIV2.1
- net Vbat: now also R_VDIV1_2.2
- new net: R_VDIV1_1.2, R_VDIV1_2.1
Changed lines of the file:
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@@
   (junction (at 135.89 106.68) (diameter 0) (color 0 0 0 0)
+  )
+  (junction (at 205.74 73.66) (diameter 0) (color 0 0 0 0)
+  )
+  (junction (at 205.74 81.28) (diameter 0) (color 0 0 0 0)
   )
   (junction (at 121.92 72.39) (diameter 0) (color 0 0 0 0)
@@
     (stroke (width 0) (type default) (color 0 0 0 0))
   )
+  (wire (pts (xy 205.74 73.66) (xy 205.74 81.28))
+    (stroke (width 0) (type default) (color 0 0 0 0))
+  )
   (wire (pts (xy 127 106.68) (xy 118.11 106.68))
     (stroke (width 0) (type default) (color 0 0 0 0))
@@
     (effects (font (size 1.27 1.27)) (justify left bottom))
   )
+  (label "Vbat" (at 205.74 58.42 0)
+    (effects (font (size 1.27 1.27)) (justify left bottom))
+  )
   (symbol (lib_id "power:GND") (at 105.41 78.74 180) (unit 1)
     (in_bom yes) (on_board yes)
@@
     (property "Reference" "L_bst1" (id 0) (at 83.82 86.614 90))
     (property "Value" "22uH" (id 1) (at 83.82 88.9254 90))
-    (property "Footprint" "Inductor_SMD:L_Wuerth_MAPI-3015" (id 2) (at 83.82 91.44 0)
+    (property "Footprint" "Inductor_SMD:L_Taiyo-Yuden_NR-30xx_HandSoldering" (id 2) (at 83.82 91.44 0)
       (effects (font (size 1.27 1.27)) hide)
     )
@@
     (pin "1")
     (pin "2")
-  )
-  (symbol (lib_id "Device:R") (at 80.01 113.03 180) (unit 1)
-    (in_bom yes) (on_board yes)
-    (property "Reference" "R_pulldown1" (id 0) (at 78.232 114.1984 0)
-      (effects (font (size 1.27 1.27)) (justify left))
-    )
-    (property "Value" "10M" (id 1) (at 78.232 111.887 0)
-      (effects (font (size 1.27 1.27)) (justify left))
-    )
-    (property "Footprint" "Resistor_SMD:R_0603_1608Metric_Pad1.05x0.95mm_HandSolder" (id 2) (at 81.788 113.03 90)
-      (effects (font (size 1.27 1.27)) hide)
-    )
-    (property "Datasheet" "~" (id 3) (at 80.01 113.03 0)
-      (effects (font (size 1.27 1.27)) hide)
-    )
-    (pin "1")
-    (pin "2")
-  )
-  (symbol (lib_id "power:GND") (at 80.01 116.84 0) (unit 1)
-    (in_bom yes) (on_board yes)
-    (property "Reference" "#PWR0102" (id 0) (at 80.01 123.19 0)
-      (effects (font (size 1.27 1.27)) hide)
-    )
-    (property "Value" "GND" (id 1) (at 80.137 121.2342 0))
-    (property "Footprint" "" (id 2) (at 80.01 116.84 0)
-      (effects (font (size 1.27 1.27)) hide)
-    )
-    (property "Datasheet" "" (id 3) (at 80.01 116.84 0)
-      (effects (font (size 1.27 1.27)) hide)
-    )
-    (pin "1")
   )
   (symbol (lib_id "Battery_Management:BQ25570") (at 102.87 104.14 0) (unit 1)
@@
     (property "Reference" "L_bst2" (id 0) (at 121.92 86.614 90))
     (property "Value" "10uH" (id 1) (at 121.92 88.9254 90))
-    (property "Footprint" "Inductor_SMD:L_Wuerth_MAPI-3015" (id 2) (at 121.92 91.44 0)
+    (property "Footprint" "Inductor_SMD:L_Taiyo-Yuden_NR-30xx_HandSoldering" (id 2) (at 121.92 91.44 0)
       (effects (font (size 1.27 1.27)) hide)
     )
@@
     )
     (property "Datasheet" "~" (id 3) (at 167.64 60.96 0)
+      (effects (font (size 1.27 1.27)) hide)
+    )
+    (pin "1")
+    (pin "2")
+  )
+  (symbol (lib_id "Device:R") (at 209.55 73.66 90) (mirror x) (unit 1)
+    (in_bom yes) (on_board yes)
+    (property "Reference" "R_VDIV2" (id 0) (at 209.55 71.12 90))
+    (property "Value" "9M" (id 1) (at 209.55 70.7136 90)
+      (effects (font (size 1.27 1.27)) hide)
+    )
+    (property "Footprint" "Resistor_SMD:R_0603_1608Metric_Pad0.98x0.95mm_HandSolder" (id 2) (at 209.55 71.882 90)
+      (effects (font (size 1.27 1.27)) hide)
+    )
+    (property "Datasheet" "~" (id 3) (at 209.55 73.66 0)
+      (effects (font (size 1.27 1.27)) hide)
+    )
+    (pin "1")
+    (pin "2")
+  )
+  (symbol (lib_id "Device:R") (at 205.74 62.23 0) (mirror x) (unit 1)
+    (in_bom yes) (on_board yes)
+    (property "Reference" "R_VDIV1_2" (id 0) (at 203.2 62.23 90))
+    (property "Value" "10M" (id 1) (at 202.7936 62.23 90)
+      (effects (font (size 1.27 1.27)) hide)
+    )
+    (property "Footprint" "Resistor_SMD:R_0603_1608Metric_Pad0.98x0.95mm_HandSolder" (id 2) (at 203.962 62.23 90)
+      (effects (font (size 1.27 1.27)) hide)
+    )
+    (property "Datasheet" "~" (id 3) (at 205.74 62.23 0)
+      (effects (font (size 1.27 1.27)) hide)
+    )
+    (pin "1")
+    (pin "2")
+  )
+  (symbol (lib_id "Device:R") (at 205.74 69.85 0) (mirror x) (unit 1)
+    (in_bom yes) (on_board yes)
+    (property "Reference" "R_VDIV1_1" (id 0) (at 203.2 69.85 90))
+    (property "Value" "8.5M" (id 1) (at 202.7936 69.85 90)
+      (effects (font (size 1.27 1.27)) hide)
+    )
+    (property "Footprint" "Resistor_SMD:R_0603_1608Metric_Pad0.98x0.95mm_HandSolder" (id 2) (at 203.962 69.85 90)
+      (effects (font (size 1.27 1.27)) hide)
+    )
+    (property "Datasheet" "~" (id 3) (at 205.74 69.85 0)
       (effects (font (size 1.27 1.27)) hide)
     )
@@
     (pin "8")
   )
+  (symbol (lib_id "power:GND") (at 213.36 73.66 0) (unit 1)
+    (in_bom yes) (on_board yes) (fields_autoplaced)
+    (property "Reference" "#PWR?" (id 0) (at 213.36 80.01 0)
+      (effects (font (size 1.27 1.27)) hide)
+    )
+    (property "Value" "GND" (id 1) (at 213.36 78.1034 0))
+    (property "Footprint" "" (id 2) (at 213.36 73.66 0)
+      (effects (font (size 1.27 1.27)) hide)
+    )
+    (property "Datasheet" "" (id 3) (at 213.36 73.66 0)
+      (effects (font (size 1.27 1.27)) hide)
+    )
+    (pin "1")
+  )
   (sheet_instances
     (path "/" (page "1"))
@@
       (reference "#PWR0101") (unit 1) (value "GND") (footprint "")
     )
-    (path "/00000000-0000-0000-0000-000061c28559"
-      (reference "#PWR0102") (unit 1) (value "GND") (footprint "")
-    )
     (path "/00000000-0000-0000-0000-000062b11626"
       (reference "#PWR0103") (unit 1) (value "GND") (footprint "")
@@
       (reference "#PWR0109") (unit 1) (value "GND") (footprint "")
     )
+    (path "/db0d2e2b-5d09-4c33-981b-9463e2497cef"
+      (reference "#PWR?") (unit 1) (value "GND") (footprint "")
+    )
     (path "/00000000-0000-0000-0000-000061c12816"
       (reference "C_Stor1") (unit 1) (value "22uF") (footprint "Capacitor_SMD:C_0805_2012Metric_Pad1.18x1.45mm_HandSolder")
@@
     )
     (path "/00000000-0000-0000-0000-0000609cfca3"
-      (reference "L_bst1") (unit 1) (value "22uH") (footprint "Inductor_SMD:L_Wuerth_MAPI-3015")
+      (reference "L_bst1") (unit 1) (value "22uH") (footprint "Inductor_SMD:L_Taiyo-Yuden_NR-30xx_HandSoldering")
     )
     (path "/00000000-0000-0000-0000-000062be4b4d"
-      (reference "L_bst2") (unit 1) (value "10uH") (footprint "Inductor_SMD:L_Wuerth_MAPI-3015")
+      (reference "L_bst2") (unit 1) (value "10uH") (footprint "Inductor_SMD:L_Taiyo-Yuden_NR-30xx_HandSoldering")
     )
     (path "/00000000-0000-0000-0000-000062d85c62"
@@
       (reference "R_LED3") (unit 1) (value "500") (footprint "Resistor_SMD:R_0603_1608Metric_Pad0.98x0.95mm_HandSolder")
     )
+    (path "/9609577c-f5d3-4fa9-b23b-517cff5b9d00"
+      (reference "R_VDIV1_1") (unit 1) (value "8.5M") (footprint "Resistor_SMD:R_0603_1608Metric_Pad0.98x0.95mm_HandSolder")
+    )
+    (path "/9100e9f7-87a2-4552-b03f-548c9b98d4a7"
+      (reference "R_VDIV1_2") (unit 1) (value "10M") (footprint "Resistor_SMD:R_0603_1608Metric_Pad0.98x0.95mm_HandSolder")
+    )
+    (path "/10d29fd5-1d93-4874-98e7-a1d59cfef03f"
+      (reference "R_VDIV2") (unit 1) (value "9M") (footprint "Resistor_SMD:R_0603_1608Metric_Pad0.98x0.95mm_HandSolder")
+    )
     (path "/00000000-0000-0000-0000-000060a15444"
       (reference "R_ok1") (unit 1) (value "3.3M") (footprint "Resistor_SMD:R_0603_1608Metric_Pad1.05x0.95mm_HandSolder")
@@
       (reference "R_ov2") (unit 1) (value "3.3M") (footprint "Resistor_SMD:R_0603_1608Metric_Pad1.05x0.95mm_HandSolder")
     )
-    (path "/00000000-0000-0000-0000-000061c260a2"
-      (reference "R_pulldown1") (unit 1) (value "10M") (footprint "Resistor_SMD:R_0603_1608Metric_Pad1.05x0.95mm_HandSolder")
-    )
     (path "/00000000-0000-0000-0000-000060a52db8"
