File: 0.3/Hardware/PCB_0.3.1/Omamori.kicad_pcb (KiCad board)
At the start: 2 copper layers, 25 x 35 mm, 35 parts, among them J1 Conn_01x03_Female, J2 Conn_01x07_Female, U1 BQ25570, U2 ATtiny1626, U3 TS-1233

Commit message: HW Update before going to germany.
Parts:
- moved C_uC_Filter4 11.0 mm to (35.1, 42.9), turned to -90 degrees
- moved R_VDIV1_2 6.39 mm to (32.3, 13.9), turned to 0 degrees
- moved R_Reset1 3.85 mm to (18.4, 17.9)
- moved C_Stor1 2.29 mm to (29.4, 16.2), turned to 180 degrees
- moved C_uC_Filter2 2.26 mm to (22.4, 25.2), turned to -90 degrees
- moved R_VDIV1_1 1.95 mm to (29.2, 13.9), turned to 0 degrees
- moved U3 1.38 mm to (18.1, 15.3)
- moved C_ref1 1.30 mm to (34.4, 24.5), turned to -90 degrees
- moved C_filter1 1.27 mm to (29.5, 18.9), turned to 180 degrees
- moved C_filter2 0.67 mm to (29.5, 17.8), turned to 180 degrees
- moved C_uC_Filter3 0.55 mm to (20.5, 24.2), turned to 90 degrees
- moved C_super1 0.15 mm to (25.0, 37.1)
Connections:
- C_Stor1 pad 1: /Vbat -> /Vstor
- C_filter1 pad 1: /Vbat -> /Vstor
- C_filter2 pad 1: /Vbat -> /Vstor
- U1 pad 19: /Vbat -> /Vstor
- U1 pad 3: /Vbat -> /Vstor
Routing:
- net GND: track 281.7 -> 339.8 mm, vias 7 -> 8
- net /Vstor: track 0.00 -> 21.2 mm, vias 0 -> 2
- net /Vbat: track 63.9 -> 46.5 mm
- net Net-(C_Reset1-Pad1): track 9.45 -> 5.94 mm
- net /Vcc_ATTiny: track 48.7 -> 45.3 mm
- net /Interrupt: track 4.01 -> 2.11 mm
- net Net-(R_VDIV1_1-Pad1): track 18.9 -> 17.6 mm
- net Net-(C_ref1-Pad1): track 2.59 -> 3.27 mm

Commit message: Updated Omamori 0.3.1.
Parts:
- removed R_Reset1: 10M, Resistor_SMD:R_0603_1608Metric_Pad0.98x0.95mm_HandSolder
- J2: value Conn_01x07_Female -> Conn_01x02_Pin; footprint Connector_PinHeader_2.54mm:PinHeader_1x07_P2.54mm_Vertical -> Connector_PinHeader_2.54mm:PinHeader_1x02_P2.54mm_Vertical; moved to B.Cu
- L_bst1: value 22uH -> LPS4018-223M 22uH
- L_bst2: value 10uH -> LPS4018-103M 10uH
- R_VDIV1_1: value 8.5M -> 8.2M
- R_VDIV2: value 9M -> 8.2M
- R_ok1: value 6.29M -> 6.2M
- R_ok2: value 3M -> 4.3M
- R_ok3: value 3.71M -> 2.4M
- R_out1: value 8.74M -> 9.1M
- R_out2: value 4.26M -> 4.7M
- R_ov1: value 4.29M -> 4.7M
- R_ov2: value 8.71M -> 9.1M
- moved J2 17.1 mm to (17.6, 27.9), turned to 0 degrees
- turned C_Reset1 to -90 degrees
Connections:
- C_Reset1 pad 1: Net-(C_Reset1-Pad1) -> GND
- C_Reset1 pad 2: GND -> /Interrupt
- J2 pad 1: GND -> Net-(J2-Pin_1)
- J2 pad 2: /Vcc_ATTiny -> Net-(J2-Pin_2)
- U2 pad 1: Net-(C_Reset1-Pad1) -> /Interrupt
- U2 pad 10: Net-(J2-Pad5) -> unconnected-(U2-PB4-Pad10)
- U2 pad 13: Net-(J2-Pad4) -> unconnected-(U2-PB1-Pad13)
- U2 pad 14: Net-(J2-Pad3) -> unconnected-(U2-PB0-Pad14)
- U2 pad 7: Net-(J2-Pad7) -> Net-(J2-Pin_2)
- U2 pad 8: unconnected-(U2-Pad8) -> Net-(J2-Pin_1)
- U2 pad 9: Net-(J2-Pad6) -> unconnected-(U2-PB5-Pad9)
Routing:
- net Net-(J2-Pad7): track 29.8 -> 0.00 mm
- net Net-(J2-Pad6): track 29.1 -> 0.00 mm
- net Net-(J2-Pad4): track 28.0 -> 0.00 mm
- net Net-(J2-Pad3): track 27.7 -> 0.00 mm
- net Net-(J2-Pad5): track 26.6 -> 0.00 mm
- net /Vcc_ATTiny: track 45.3 -> 26.1 mm
- net GND: track 339.8 -> 347.0 mm
- net /Interrupt: track 2.11 -> 8.28 mm
- net Net-(J2-Pin_1): track 0.00 -> 5.98 mm
- net Net-(C_Reset1-Pad1): track 5.94 -> 0.00 mm
- net Net-(U2-PA1): track 17.6 -> 22.6 mm
- net Net-(Sol_1-GND): track 46.8 -> 51.3 mm
- net Net-(J2-Pin_2): track 0.00 -> 2.72 mm
- net Net-(J1-Pin_2): track 13.1 -> 13.7 mm
Other:
- board text added: "P"
- board text removed: "D"
