File: 0.3/Hardware/PCB_0.3.1/Omamori.kicad_sch (KiCad schematic)
At the start: 34 parts, among them J1 Conn_01x03_Female, J2 Conn_01x07_Female, U1 BQ25570, U2 ATtiny1626, U3 TS-1233

Commit message: HW Update before going to germany.
Connections:
- net Vbat: no longer C_Stor1.1, C_filter1.1, C_filter2.1, U1.19 (VSTOR), U1.3 (VOC_SAMP)
- new net Vstor: C_Stor1.1, C_filter1.1, C_filter2.1, U1.19 (VSTOR), U1.3 (VOC_SAMP)
Changed lines of the file:
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@@
   (junction (at 144.78 102.87) (diameter 0) (color 0 0 0 0)
-  )
-  (junction (at 102.87 60.96) (diameter 0) (color 0 0 0 0)
   )
   (junction (at 134.62 128.27) (diameter 0) (color 0 0 0 0)
@@
   )
   (junction (at 72.39 80.01) (diameter 0) (color 0 0 0 0)
-  )
-  (junction (at 105.41 60.96) (diameter 0) (color 0 0 0 0)
   )
   (junction (at 167.64 85.09) (diameter 0) (color 0 0 0 0)
@@
     (stroke (width 0) (type default) (color 0 0 0 0))
   )
-  (wire (pts (xy 102.87 60.96) (xy 105.41 60.96))
-    (stroke (width 0) (type default) (color 0 0 0 0))
-  )

Commit message: Updated Omamori 0.3.1.
Parts:
- removed J2: Conn_01x07_Female, Connector_PinHeader_2.54mm:PinHeader_1x07_P2.54mm_Vertical, symbol Connector:Conn_01x07_Female
- removed R_Reset1: 10M, Resistor_SMD:R_0603_1608Metric_Pad0.98x0.95mm_HandSolder, symbol Device:R
- added J2: Conn_01x02_Pin, Connector_PinHeader_2.54mm:PinHeader_1x02_P2.54mm_Vertical, symbol Connector:Conn_01x02_Pin
- L_bst1: value 22uH -> LPS4018-223M 22uH
- L_bst2: value 10uH -> LPS4018-103M 10uH
- R_VDIV1_1: value 8.5M -> 8.2M
- R_VDIV2: value 9M -> 8.2M
- R_ok1: value 6.29M -> 6.2M
- R_ok2: value 3M -> 4.3M
- R_ok3: value 3.71M -> 2.4M
- R_out1: value 8.74M -> 9.1M
- R_out2: value 4.26M -> 4.7M
- R_ov1: value 4.29M -> 4.7M
- R_ov2: value 8.71M -> 9.1M
Connections:
- net GND: now also C_Reset1.1; no longer C_Reset1.2
- net Interrupt: now also C_Reset1.2, U2.1 (PA2)
- net at U2.7 (PA6): now also J2.2 (Pin_2)
- net at U2.8 (PA7): now also J2.1 (Pin_1)
- no-connect marks 9 -> 12
Other:
- company: (none) -> Felix Mark
- title: (none) -> Omamori
- moved on the sheet: C_Reset1, C_Stor1, C_filter1, C_filter2, C_hvr1, C_ref1, C_super1, C_uC_Filter1, C_uC_Filter2, C_uC_Filter3, C_uC_Filter4, D1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
